Commit message: real_tool tool_end frames added

File: robothon2023_cell/robothon2023_description/urdf/sharework_cell.urdf.xacro (robot description, xacro)
@@ -291,4 +291,16 @@
   />
 </xacro:if>
+<joint name="flage_to_real_tool" type="fixed">
+  <parent link="tool0" />
+  <child link = "real_tool" />
+  <origin xyz="0.0 0.0 0.149" rpy="0 0 0" />
+</joint>
+<link name="real_tool"/>
+<joint name="flage_to_tool_end" type="fixed">
+  <parent link="tool0" />
+  <child link = "tool_end" />
+  <origin xyz="0.0 0.0 0.149" rpy="0 0 0" />
+</joint>
+<link name="tool_end"/>
 <joint name="cursor_to_base" type="fixed">
   <parent link="cursor" />

Commit message: Advancement

File: robothon2023_cell/robothon2023_description/urdf/sharework_cell.urdf.xacro (robot description, xacro)
@@ -297,8 +297,14 @@
 </joint>
 <link name="real_tool"/>
+<joint name="real_tool_to_door" type="fixed">
+  <parent link="tool_end" />
+  <child link = "door" />
+  <origin xyz="0.0 0.04 0.04" rpy="0 0 0" />
+</joint>
+<link name="door"/>
 <joint name="flage_to_tool_end" type="fixed">
   <parent link="tool0" />
   <child link = "tool_end" />
-  <origin xyz="0.0 0.0 0.149" rpy="0 0 0" />
+  <origin xyz="0.0 0.0 0.180" rpy="0 0 0" />
 </joint>
 <link name="tool_end"/>
